Commit message: fixed bug

File: lunabot_description/urdf/lunabot_ros2_control.xacro (robot description, xacro)
@@ -1,15 +1,25 @@
 <?xml version="1.0"?>
 <robot xmlns:xacro="http://www.ros.org/wiki/xacro">
-  <ros2_control name="MobileBaseHardwareInterface" type="system">
+  <ros2_control name="LunabotHardwareInterface" type="system">
     <hardware>
       <plugin>mock_components/GenericSystem</plugin>
       <param name="calculate_dynamics">true</param>
     </hardware>
-    <joint name="base_right_wheel_joint">
+    <joint name="front_left_wheel">
       <command_interface name="velocity"/>
       <state_interface name="position"/>
       <state_interface name="velocity"/>
     </joint>
-    <joint name="base_left_wheel_joint">
+    <joint name="rear_left_wheel">
+      <command_interface name="velocity"/>
+      <state_interface name="position"/>
+      <state_interface name="velocity"/>
+    </joint>
+    <joint name="front_right_wheel">
+      <command_interface name="velocity"/>
+      <state_interface name="position"/>
+      <state_interface name="velocity"/>
+    </joint>
+    <joint name="rear_right_wheel">
       <command_interface name="velocity"/>
       <state_interface name="position"/>
