Commit message: Add lift and tilt assembly to URDF

File: lunabot_description/urdf/lunabot_core.xacro (robot description, xacro)
@@ -99,3 +99,100 @@
     <!-- Rear Right -->
     <xacro:wheel name="rear_right_wheel"  x="-0.35" y="-0.325" z="0"/>
+    <!-- ===============================
+         LIFT + BUCKET ASSEMBLY
+         Simplified representation of the
+         lift arm, bucket, and actuators.
+         =============================== -->
+    <joint name="lift_joint" type="revolute">
+        <parent link="chassis"/>
+        <child link="lift_arm"/>
+        <!-- Lift pivot near the front-top of chassis -->
+        <origin xyz="0.3 0 0.15" rpy="0 0 0"/>
+        <axis xyz="0 1 0"/>
+        <limit lower="-0.5" upper="1.2" effort="200" velocity="1.0"/>
+    </joint>
+    <link name="lift_arm">
+        <visual>
+            <geometry>
+                <box size="0.6 0.15 0.1"/>
+            </geometry>
+            <material name="blue"/>
+        </visual>
+        <collision>
+            <geometry>
+                <box size="0.6 0.15 0.1"/>
+            </geometry>
+        </collision>
+        <xacro:inertial_box mass="6.0" x="0.6" y="0.15" z="0.1">
+            <origin xyz="0.15 0 0.05" rpy="0 0 0"/>
+        </xacro:inertial_box>
+    </link>
+    <joint name="bucket_joint" type="revolute">
+        <parent link="lift_arm"/>
+        <child link="bucket"/>
+        <!-- Bucket hinge at front of arm -->
+        <origin xyz="0.3 0 0.05" rpy="0 0 0"/>
+        <axis xyz="0 1 0"/>
+        <limit lower="-1.2" upper="0.8" effort="150" velocity="1.0"/>
+    </joint>
+    <link name="bucket">
+        <visual>
+            <geometry>
+                <box size="0.35 0.4 0.2"/>
+            </geometry>
+            <material name="white"/>
+        </visual>
+        <collision>
+            <geometry>
+                <box size="0.35 0.4 0.2"/>
+            </geometry>
+        </collision>
+        <xacro:inertial_box mass="4.0" x="0.35" y="0.4" z="0.2">
+            <origin xyz="0 0 0" rpy="0 0 0"/>
+        </xacro:inertial_box>
+    </link>
+    <!-- Lift actuator (visual only) -->
+    <joint name="lift_actuator_joint" type="fixed">
+        <parent link="chassis"/>
+        <child link="lift_actuator"/>
+        <origin xyz="0.1 0 0.1" rpy="0 ${pi/2} 0"/>
+    </joint>
+    <link name="lift_actuator">
+        <visual>
+            <geometry>
+                <cylinder radius="0.03" length="0.45"/>
+            </geometry>
+            <material name="black"/>
+        </visual>
+        <collision>
+            <geometry>
+                <cylinder radius="0.03" length="0.45"/>
+            </geometry>
+        </collision>
+        <xacro:inertial_cylinder mass="1.0" length="0.45" radius="0.03">
+            <origin xyz="0 0 0" rpy="0 0 0"/>
+        </xacro:inertial_cylinder>
+    </link>
+    <!-- Tilt actuator (visual only) -->
+    <joint name="tilt_actuator_joint" type="fixed">
+        <parent link="lift_arm"/>
+        <child link="tilt_actuator"/>
+        <origin xyz="0.2 0 -0.05" rpy="0 ${pi/2} 0"/>
+    </joint>
+    <link name="tilt_actuator">
+        <visual>
+            <geometry>
+                <cylinder radius="0.025" length="0.3"/>
+            </geometry>
+            <material name="black"/>
+        </visual>
+        <collision>
+            <geometry>
+                <cylinder radius="0.025" length="0.3"/>
+            </geometry>
+        </collision>
+        <xacro:inertial_cylinder mass="0.6" length="0.3" radius="0.025">
+            <origin xyz="0 0 0" rpy="0 0 0"/>
+        </xacro:inertial_cylinder>
+    </link>
 </robot>
